File: PCB/megadesk.kicad_pcb (KiCad board)
At the start: 2 copper layers, 42.2 x 32.8 mm, 20 parts, among them J1 Interface, J2 FFC, J3 AVR-ISP-6, U1 L7812, U2 L7805, U3 ATTINY841-SSU, U4 MCP2003B

Commit message: Coredump adjustments
Other:
- board text added: "coredump.ch edition"
- board text added: "github.com/gcormier/megadesk"
- board text removed: "JLCJLCJLCJLC"
